File: Computer.kicad_pcb (KiCad board)
At the start: 2 copper layers, 54 parts, among them J1 DB9, J2 Screw_Terminal_1x04, U1 8284, U10 74LS04, U11 7400, U12 8259, U13 74LS138, U14 LM7905CT, U15 LM7912CT, U16 MAX202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

Commit message: Added edge cuts
Other:
- board outline added: 147.3 x 128.3 mm
Changed lines of the file:
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@@
     (area 37.624999 29.109999 189.5316 157.580001)
     (thickness 1.6)
-    (drawings 12)
+    (drawings 16)
     (tracks 1665)
     (zones 0)
@@
       (net 20 A0))
   )
+  (gr_line (start 41.91 157.48) (end 41.91 29.21) (layer Edge.Cuts) (width 0.1))
+  (gr_line (start 189.23 157.48) (end 41.91 157.48) (layer Edge.Cuts) (width 0.1))
+  (gr_line (start 189.23 29.21) (end 189.23 157.48) (layer Edge.Cuts) (width 0.1))
+  (gr_line (start 41.91 29.21) (end 189.23 29.21) (layer Edge.Cuts) (width 0.1))
   (gr_circle (center 185.42 153.67) (end 184.15 152.4) (layer F.SilkS) (width 0.2))
   (gr_circle (center 45.72 153.67) (end 46.99 152.4) (layer F.SilkS) (width 0.2))
